File: KiCAD/BS112.kicad_sch (KiCad schematic)
At the start: 3 parts

Commit message: Connections finished
Connections:
- net 501 renamed 501 SWB Motor
- net 502 renamed 502 SWA Motor
- net 507 renamed 507 Com
- net 508 renamed 508 LA Netz
- net 509 renamed 509 LA Motor
Changed lines of the file:
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@@
     (stroke (width 0) (type default) (color 0 0 0 0))
   )
-  (hierarchical_label "502" (shape input) (at 146.05 78.74 90)
+  (hierarchical_label "502 SWA Motor" (shape passive) (at 146.05 78.74 90)
     (effects (font (size 1.27 1.27)) (justify left))
   )
-  (hierarchical_label "503" (shape input) (at 152.4 105.41 270)
+  (hierarchical_label "503 SWB Motor" (shape passive) (at 152.4 105.41 270)
     (effects (font (size 1.27 1.27)) (justify right))
   )
-  (hierarchical_label "507" (shape input) (at 123.19 105.41 270)
+  (hierarchical_label "507 Com" (shape input) (at 123.19 105.41 270)
     (effects (font (size 1.27 1.27)) (justify right))
   )
-  (hierarchical_label "501" (shape input) (at 146.05 105.41 270)
+  (hierarchical_label "501 SWB Motor" (shape passive) (at 146.05 105.41 270)
     (effects (font (size 1.27 1.27)) (justify right))
   )
-  (hierarchical_label "509" (shape input) (at 129.54 78.74 90)
+  (hierarchical_label "509 LA Motor" (shape input) (at 129.54 78.74 90)
     (effects (font (size 1.27 1.27)) (justify left))
   )
-  (hierarchical_label "508" (shape input) (at 116.84 78.74 90)
+  (hierarchical_label "508 LA Netz" (shape input) (at 116.84 78.74 90)
     (effects (font (size 1.27 1.27)) (justify left))
   )

Commit message: Labels
Parts:
- LA1: value (none) -> Netz
- LA2, SW1: value (none) -> Motor
Changed lines of the file:
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@@
       (effects (font (size 1.27 1.27)) (justify left))
     )
-    (property "Value" "" (id 1) (at 132.715 94.4122 0)
+    (property "Value" "Motor" (id 1) (at 132.715 94.4122 0)
       (effects (font (size 1.27 1.27)) (justify left))
     )
@@
       (effects (font (size 1.27 1.27)) (justify left))
     )
-    (property "Value" "" (id 1) (at 120.015 94.4122 0)
+    (property "Value" "Netz" (id 1) (at 120.015 94.4122 0)
       (effects (font (size 1.27 1.27)) (justify left))
     )
@@
       (effects (font (size 1.27 1.27)) (justify right))
     )
-    (property "Value" "" (id 1) (at 147.193 94.4122 90)
+    (property "Value" "Motor" (id 1) (at 147.193 94.4122 90)
       (effects (font (size 1.27 1.27)) (justify right))
     )
