File: KiCAD/BS263.kicad_sch (KiCad schematic)
At the start: 33 parts

Commit message: Connections finished
Parts:
- gave numbers to parts that had none: 1
Connections:
- net 1 renamed 1 0V
- net 16 renamed 16 +10V
- net 18 renamed 18 K1B
- net 19 renamed 19 K1A
- net 2 renamed 2 Start Btn
- net 21 renamed 21 K2B
- net 22 renamed 22 K2A
- net 23 renamed 23 18VAC
- net 24 renamed 24 18VAC
- net 25 renamed 25 +24V
- net 3 renamed 3 Auto Start
- net 8 renamed 8 -10V
Other:
- moved on the sheet: C8, D8, R10

Commit message: Labels
Parts:
- C4: value (none) -> 1u
- C8: value (none) -> 470n
- D1, D2, D3, D4, D8, D9: value (none) -> ZS70
- D5: value (none) -> BZY88
- D6, D7: value (none) -> DD006
- F1, F2: value (none) -> 1.5A
- K1: value (none) -> DIPxx-2Axx-21x; footprint (none) -> Relay_THT:Relay_StandexMeder_DIP_LowProfile
- Q1, Q2, Q3, Q4, Q5: value (none) -> BFY51
- R1, R3, R7: value (none) -> 10k
- R10: value (none) -> 10
- R2: value (none) -> 33k
- R4: value (none) -> 4k7
- R5: value (none) -> 470
- R6: value (none) -> 47
- R8: value (none) -> 2k2
- R9: value (none) -> 22k
Changed lines of the file:
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@@
     (in_bom yes) (on_board yes)
     (property "Reference" "D6" (id 0) (at 208.28 64.77 0))
-    (property "Value" "" (id 1) (at 207.01 67.31 0))
+    (property "Value" "DD006" (id 1) (at 207.01 67.31 0))
     (property "Footprint" "" (id 2) (at 213.36 68.58 0)
       (effects (font (size 1.27 1.27)) hide)
@@
     (in_bom yes) (on_board yes)
     (property "Reference" "D7" (id 0) (at 208.28 69.85 0))
-    (property "Value" "" (id 1) (at 207.01 72.39 0))
+    (property "Value" "DD006" (id 1) (at 207.01 72.39 0))
     (property "Footprint" "" (id 2) (at 213.36 73.66 0)
       (effects (font (size 1.27 1.27)) hide)
@@
       (effects (font (size 1.27 1.27)) (justify left))
     )
-    (property "Value" "" (id 1) (at 203.962 102.743 90)
+    (property "Value" "ZS70" (id 1) (at 203.962 102.743 90)
       (effects (font (size 1.27 1.27)) (justify left))
     )
@@
     (in_bom yes) (on_board yes)
     (property "Reference" "D9" (id 0) (at 161.29 102.4382 0))
-    (property "Value" "" (id 1) (at 161.29 104.7496 0))
+    (property "Value" "ZS70" (id 1) (at 161.29 104.7496 0))
     (property "Footprint" "" (id 2) (at 161.29 107.95 0)
       (effects (font (size 1.27 1.27)) hide)
@@
       (effects (font (size 1.27 1.27)) (justify left))
     )
-    (property "Value" "" (id 1) (at 74.422 130.683 90)
+    (property "Value" "ZS70" (id 1) (at 74.422 130.683 90)
       (effects (font (size 1.27 1.27)) (justify left))
     )
@@
     (in_bom yes) (on_board yes)
     (property "Reference" "D1" (id 0) (at 46.99 60.5282 0))
-    (property "Value" "" (id 1) (at 46.99 62.8396 0))
+    (property "Value" "ZS70" (id 1) (at 46.99 62.8396 0))
     (property "Footprint" "" (id 2) (at 46.99 66.04 0)
       (effects (font (size 1.27 1.27)) hide)
@@
     (in_bom yes) (on_board yes)
     (property "Reference" "D2" (id 0) (at 46.99 69.4182 0))
-    (property "Value" "" (id 1) (at 46.99 71.7296 0))
+    (property "Value" "ZS70" (id 1) (at 46.99 71.7296 0))
     (property "Footprint" "" (id 2) (at 46.99 74.93 0)
       (effects (font (size 1.27 1.27)) hide)
@@
     (in_bom yes) (on_board yes)
     (property "Reference" "D3" (id 0) (at 46.99 79.5782 0))
-    (property "Value" "" (id 1) (at 46.99 81.8896 0))
+    (property "Value" "ZS70" (id 1) (at 46.99 81.8896 0))
     (property "Footprint" "" (id 2) (at 46.99 85.09 0)
       (effects (font (size 1.27 1.27)) hide)
@@
     (in_bom yes) (on_board yes)
     (property "Reference" "D5" (id 0) (at 58.42 79.5782 0))
-    (property "Value" "" (id 1) (at 58.42 81.8896 0))
+    (property "Value" "BZY88" (id 1) (at 58.42 81.8896 0))
     (property "Footprint" "" (id 2) (at 58.42 85.09 0)
       (effects (font (size 1.27 1.27)) hide)
@@
       (effects (font (size 1.27 1.27)) (justify left) hide)
     )
-    (property "Value" "" (id 1) (at 227.33 70.993 90))
+    (property "Value" "1.5A" (id 1) (at 227.33 70.993 90))
     (property "Footprint" "" (id 2) (at 227.33 75.438 90)
       (effects (font (size 1.27 1.27)) hide)
@@
       (effects (font (size 1.27 1.27)) hide)
     )
-    (property "Value" "" (id 1) (at 227.33 65.913 90))
+    (property "Value" "1.5A" (id 1) (at 227.33 65.913 90))
     (property "Footprint" "" (id 2) (at 227.33 70.358 90)
       (effects (font (size 1.27 1.27)) hide)
@@
       (effects (font (size 1.27 1.27)) (justify left))
     )
-    (property "Value" "" (id 1) (at 112.8014 115.443 0)
+    (property "Value" "BFY51" (id 1) (at 112.8014 115.443 0)
       (effects (font (size 1.27 1.27)) (justify left))
     )
@@
       (effects (font (size 1.27 1.27)) (justify left))
     )
-    (property "Value" "" (id 1) (at 133.1214 107.823 0)
+    (property "Value" "BFY51" (id 1) (at 133.1214 107.823 0)
       (effects (font (size 1.27 1.27)) (justify left))
     )
@@
       (effects (font (size 1.27 1.27)) (justify left))
     )
-    (property "Value" "" (id 1) (at 215.6714 124.333 0)
+    (property "Value" "BFY51" (id 1) (at 215.6714 124.333 0)
       (effects (font (size 1.27 1.27)) (justify left))
     )
@@
       (effects (font (size 1.27 1.27)) (justify left))
     )
-    (property "Value" "" (id 1) (at 154.7114 101.473 0)
+    (property "Value" "BFY51" (id 1) (at 154.7114 101.473 0)
       (effects (font (size 1.27 1.27)) (justify left))
     )
@@
       (effects (font (size 1.27 1.27)) (justify left))
     )
-    (property "Value" "" (id 1) (at 186.4614 102.743 0)
+    (property "Value" "BFY51" (id 1) (at 186.4614 102.743 0)
       (effects (font (size 1.27 1.27)) (justify left))
     )
@@
       (effects (font (size 1.27 1.27)) (justify left))
     )
-    (property "Value" "" (id 1) (at 65.278 109.093 0)
+    (property "Value" "10k" (id 1) (at 65.278 109.093 0)
       (effects (font (size 1.27 1.27)) (justify left))
     )
@@
       (effects (font (size 1.27 1.27)) (justify left))
     )
-    (property "Value" "" (id 1) (at 65.278 130.683 0)
+    (property "Value" "33k" (id 1) (at 65.278 130.683 0)
       (effects (font (size 1.27 1.27)) (justify left))
     )
@@
       (effects (font (size 1.27 1.27)) (justify left))
     )
-    (property "Value" "" (id 1) (at 97.028 106.553 0)
+    (property "Value" "10k" (id 1) (at 97.028 106.553 0)
       (effects (font (size 1.27 1.27)) (justify left))
     )
@@
       (effects (font (size 1.27 1.27)) (justify left))
     )
-    (property "Value" "" (id 1) (at 123.698 90.043 0)
+    (property "Value" "4k7" (id 1) (at 123.698 90.043 0)
       (effects (font (size 1.27 1.27)) (justify left))
     )
@@
       (effects (font (size 1.27 1.27)) (justify left))
     )
-    (property "Value" "" (id 1) (at 140.208 90.043 0)
+    (property "Value" "470" (id 1) (at 140.208 90.043 0)
       (effects (font (size 1.27 1.27)) (justify left))
     )
@@
       (effects (font (size 1.27 1.27)) (justify left))
     )
-    (property "Value" "" (id 1) (at 152.908 130.683 0)
+    (property "Value" "10k" (id 1) (at 152.908 130.683 0)
       (effects (font (size 1.27 1.27)) (justify left))
     )
@@
       (effects (font (size 1.27 1.27)) (justify left))
     )
-    (property "Value" "" (id 1) (at 170.688 117.983 0)
+    (property "Value" "47" (id 1) (at 170.688 117.983 0)
       (effects (font (size 1.27 1.27)) (justify left))
     )
@@
       (effects (font (size 1.27 1.27)) (justify left))
     )
-    (property "Value" "" (id 1) (at 185.928 130.683 0)
+    (property "Value" "22k" (id 1) (at 185.928 130.683 0)
       (effects (font (size 1.27 1.27)) (justify left))
     )
@@
       (effects (font (size 1.27 1.27)) (justify left))
     )
-    (property "Value" "" (id 1) (at 185.928 117.983 0)
+    (property "Value" "2k2" (id 1) (at 185.928 117.983 0)
       (effects (font (size 1.27 1.27)) (justify left))
     )
@@
       (effects (font (size 1.27 1.27)) (justify left))
     )
-    (property "Value" "" (id 1) (at 244.348 111.633 0)
+    (property "Value" "10" (id 1) (at 244.348 111.633 0)
       (effects (font (size 1.27 1.27)) (justify left))
     )
@@
       (effects (font (size 1.27 1.27)) (justify left))
     )
-    (property "Value" "" (id 1) (at 98.171 130.683 0)
+    (property "Value" "1u" (id 1) (at 98.171 130.683 0)
       (effects (font (size 1.27 1.27)) (justify left))
     )
@@
       (effects (font (size 1.27 1.27)) (justify left))
     )
-    (property "Value" "" (id 1) (at 245.491 98.933 0)
+    (property "Value" "470n" (id 1) (at 245.491 98.933 0)
       (effects (font (size 1.27 1.27)) (justify left))
     )
@@
       (effects (font (size 1.27 1.27)) (justify left) hide)
     )
-    (property "Value" "" (id 1) (at 233.172 102.743 0)
+    (property "Value" "DIPxx-2Axx-21x" (id 1) (at 233.172 102.743 0)
       (effects (font (size 1.27 1.27)) (justify left) hide)
     )
-    (property "Footprint" "" (id 2) (at 233.68 102.87 0)
+    (property "Footprint" "Relay_THT:Relay_StandexMeder_DIP_LowProfile" (id 2) (at 233.68 102.87 0)
       (effects (font (size 1.27 1.27)) (justify left) hide)
     )

Commit message: Labels added
Parts:
- C1-C3, C5, C6-C7, RV1: value ~ -> (none)
Changed lines of the file:
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@@
     (in_bom yes) (on_board yes)
     (property "Reference" "RV1" (id 0) (at 160.02 116.459 90))
-    (property "Value" "~" (id 1) (at 160.02 118.7704 90))
+    (property "Value" "" (id 1) (at 160.02 118.7704 90))
     (property "Footprint" "" (id 2) (at 160.02 124.968 90)
       (effects (font (size 1.27 1.27)) hide)
@@
     (in_bom yes) (on_board yes)
     (property "Reference" "C5" (id 0) (at 109.22 91.313 90))
-    (property "Value" "~" (id 1) (at 109.22 93.6244 90))
+    (property "Value" "" (id 1) (at 109.22 93.6244 90))
     (property "Footprint" "" (id 2) (at 105.41 98.7552 0)
       (effects (font (size 1.27 1.27)) hide)
@@
       (effects (font (size 1.27 1.27)) (justify left))
     )
-    (property "Value" "~" (id 1) (at 171.9072 130.683 0)
+    (property "Value" "" (id 1) (at 171.9072 130.683 0)
       (effects (font (size 1.27 1.27)) (justify left))
     )
@@
       (effects (font (size 1.27 1.27)) (justify left))
     )
-    (property "Value" "~" (id 1) (at 86.8172 95.123 0)
+    (property "Value" "" (id 1) (at 86.8172 95.123 0)
       (effects (font (size 1.27 1.27)) (justify left))
     )
